Commit message: commit_

File: nina_description/urdf/nina.urdf.xacro (robot description, xacro)
@@ -141,3 +141,33 @@
     <axis xyz="0 0 0" />
   </joint>
+  <link name="imu_link">
+    <inertial>
+      <origin xyz="-0.00552433659106688 0.000168210391520346 0.000514000497342681" rpy="0 0 0" />
+      <mass value="0.000528415362211671" />
+      <inertia ixx="1.46176048428261E-08" ixy="1.40015117949421E-10" ixz="-1.99633872937403E-12"
+               iyy="8.59662482954888E-09" iyz="7.52375112767959E-12"
+               izz="2.30279421279312E-08" />
+    </inertial>
+    <visual>
+      <origin xyz="0 0 0" rpy="0 0 0" />
+      <geometry>
+        <mesh filename="package://nina_description/meshes/imu_link.STL" />
+      </geometry>
+      <material name="">
+        <color rgba="0.792156862745098 0.819607843137255 0.933333333333333 1" />
+      </material>
+    </visual>
+    <collision>
+      <origin xyz="0 0 0" rpy="0 0 0" />
+      <geometry>
+        <mesh filename="package://nina_description/meshes/imu_link.STL" />
+      </geometry>
+    </collision>
+  </link>
+  <joint name="imu_joint" type="fixed">
+    <origin xyz="0 0 0.0698986241758014" rpy="0 0 0" />
+    <parent link="base_link" />
+    <child link="imu_link" />
+    <axis xyz="0 0 0" />
+  </joint>
 </robot>

File: nina_description/urdf/nina_gazebo.xacro (robot description, xacro)
@@ -60,3 +60,53 @@
     </plugin>
   </gazebo>
+  <!-- IMU -->
+  <gazebo reference="imu_link">
+    <sensor name="imu" type="imu">
+        <always_on>true</always_on>
+        <update_rate>100</update_rate>
+        <imu>
+          <angular_velocity>
+            <x>
+              <noise type="gaussian">
+                <mean>0.0</mean>
+                <stddev>2e-4</stddev>
+              </noise>
+            </x>
+            <y>
+              <noise type="gaussian">
+                <mean>0.0</mean>
+                <stddev>2e-4</stddev>
+              </noise>
+            </y>
+            <z>
+              <noise type="gaussian">
+                <mean>0.0</mean>
+                <stddev>2e-4</stddev>
+              </noise>
+            </z>
+          </angular_velocity>
+          <linear_acceleration>
+            <x>
+              <noise type="gaussian">
+                <mean>0.0</mean>
+                <stddev>1.7e-2</stddev>
+              </noise>
+            </x>
+            <y>
+              <noise type="gaussian">
+                <mean>0.0</mean>
+                <stddev>1.7e-2</stddev>
+              </noise>
+            </y>
+            <z>
+              <noise type="gaussian">
+                <mean>0.0</mean>
+                <stddev>1.7e-2</stddev>
+              </noise>
+            </z>
+          </linear_acceleration>
+        </imu>
+        <plugin name="imu" filename="libgazebo_ros_imu_sensor.so"/>
+    </sensor>
+  </gazebo>
 </robot>

File: nina_description/urdf/nina_ros2_control.xacro (robot description, xacro)
@@ -1,4 +1,4 @@
 <?xml version="1.0"?>
-<robot xmlns:xacro="http://www.ros.org/wiki/xacro" name="nina">
+<robot xmlns:xacro="http://www.ros.org/wiki/xacro" name="bumperbot">
     <ros2_control name="RobotSystem" type="system">
         <!-- ros2_control Gazebo -->

Commit message: commit

File: nina_description/urdf/nina.urdf.xacro (robot description, xacro)
@@ -171,3 +171,30 @@
     <axis xyz="0 0 0" />
   </joint>
+  <link name="laser_link">
+    <inertial>
+      <origin xyz="-0.011945780406062 -0.000381929217680526 -0.0170649378129477" rpy="0 0 0" />
+      <mass value="0.073084435549317" />
+      <inertia ixx="1.96074931730795E-05" ixy="-3.62091076640009E-07" ixz="4.28230084046735E-07"
+               iyy="2.40983835136327E-05" iyz="1.50180909250652E-08"
+               izz="4.14184164228595E-05" />
+    </inertial>
+    <visual>
+      <origin xyz="0 0 0" rpy="0 0 0" />
+      <geometry>
+        <mesh filename="package://nina_description/meshes/laser_link.STL" />
+      </geometry>
+    </visual>
+    <collision>
+      <origin xyz="0 0 0" rpy="0 0 0" />
+      <geometry>
+        <mesh filename="package://nina_description/meshes/laser_link.STL" />
+      </geometry>
+    </collision>
+  </link>
+  <joint name="laser_joint" type="fixed">
+    <origin xyz="-0.0050526 -0.0023221 0.1208" rpy="0 0 3.14" />
+    <parent link="base_link" />
+    <child link="laser_link" />
+    <axis xyz="0 0 0" />
+  </joint>
 </robot>

File: nina_description/urdf/nina_gazebo.xacro (robot description, xacro)
@@ -25,4 +25,5 @@
     <maxVel>0.1</maxVel>
     <fdir1>1 0 0</fdir1>
+    <material>Gazebo/Black</material>
   </gazebo>
   <gazebo reference="wheel_right_link">
@@ -34,4 +35,5 @@
     <maxVel>0.1</maxVel>
     <fdir1>1 0 0</fdir1>
+    <material>Gazebo/Black</material>
   </gazebo>
   <!-- Caster Wheels -->
@@ -43,4 +45,5 @@
     <minDepth>0.001</minDepth>
     <maxVel>1.0</maxVel>
+    <material>Gazebo/Black</material>
   </gazebo>
   <gazebo reference="caster_front_link">
@@ -51,4 +54,5 @@
     <minDepth>0.001</minDepth>
     <maxVel>1.0</maxVel>
+    <material>Gazebo/Black</material>
   </gazebo>
   <!-- ROS 2 Control -->
@@ -110,3 +114,39 @@
     </sensor>
   </gazebo>
+    <!-- 2D Laser Sensor -->
+    <gazebo reference="laser_link">
+      <sensor name="lidar" type="ray">
+        <always_on>true</always_on>
+        <visualize>true</visualize>
+        <update_rate>5</update_rate>
+        <ray>
+          <scan>
+            <horizontal>
+              <samples>360</samples>
+              <resolution>1.00000</resolution>
+              <min_angle>0.000000</min_angle>
+              <max_angle>6.280000</max_angle>
+            </horizontal>
+          </scan>
+          <range>
+            <min>0.120000</min>
+            <max>12.0</max>
+            <resolution>0.02</resolution>
+          </range>
+          <noise>
+            <type>gaussian</type>
+            <mean>0.0</mean>
+            <stddev>0.01</stddev>
+          </noise>
+        </ray>
+        <plugin name="scan" filename="libgazebo_ros_ray_sensor.so">
+          <ros>
+            <remapping>~/out:=scan</remapping>
+          </ros>
+          <output_type>sensor_msgs/LaserScan</output_type>
+          <frame_name>laser_link</frame_name>
+        </plugin>
+      </sensor>
+      <material>Gazebo/Black</material>
+    </gazebo>
 </robot>

Commit message: adding_ig_gz

File: nina_description/urdf/nina.urdf.xacro (robot description, xacro)
@@ -1,8 +1,11 @@
 <?xml version="1.0"?>
 <robot name="nina" xmlns:xacro="http://ros.org/wiki/xacro">
+  <xacro:arg name="is_ignition" default="true"/>
   <!-- Include Gazebo Parameters -->
-  <xacro:include filename="$(find nina_description)/urdf/nina_gazebo.xacro" />
+  <!-- xacro:include filename="$(find nina_description)/urdf/nina_gazebo.xacro" /-->
+  <xacro:include filename="$(find nina_description)/urdf/nina_is_gazebo.xacro" />
+  <xacro:include filename="$(find nina_description)/urdf/nina_ros2_control_ign.xacro" />
   <!-- Include ros2_control Plugins -->
-  <xacro:include filename="$(find nina_description)/urdf/nina_ros2_control.xacro" />
+  <!-- <xacro:include filename="$(find nina_description)/urdf/nina_ros2_control.xacro" /> -->
   <link name="base_footprint"/>
   <link name="base_link">
@@ -184,4 +187,7 @@
         <mesh filename="package://nina_description/meshes/laser_link.STL" />
       </geometry>
+      <!-- <material name="">
+        <color rgba="0.792156862745098 0.819607843137255 0.933333333333333 1" />
+      </material> -->
     </visual>
     <collision>

File: nina_description/urdf/nina_gazebo.xacro (robot description, xacro)
@@ -2,5 +2,5 @@
 <robot name="nina" xmlns:xacro="http://ros.org/wiki/xacro">
   <!-- Move this one to ros2 control -->
-  <transmission name="wheel_right_transmission">
+  <!-- <transmission name="wheel_right_transmission">
     <plugin>transmission_interface/SimpleTransmission</plugin>
     <actuator name="wheel_right_motor" role="actuator_right"/>
@@ -15,5 +15,5 @@
       <mechanical_reduction>1.0</mechanical_reduction>
     </joint>
-  </transmission>
+  </transmission> -->
   <!-- Wheels -->
   <gazebo reference="wheel_left_link">
@@ -57,5 +57,5 @@
   </gazebo>
   <!-- ROS 2 Control -->
-  <gazebo>
+  <!-- <gazebo>
     <plugin filename="libgazebo_ros2_control.so" name="gazebo_ros2_control">
       <robot_param>robot_description</robot_param>
@@ -63,7 +63,7 @@
       <parameters>$(find nina_controller)/config/nina_controllers.yaml</parameters>
     </plugin>
-  </gazebo>
+  </gazebo> -->
   <!-- IMU -->
-  <gazebo reference="imu_link">
+  <!-- <gazebo reference="imu_link">
     <sensor name="imu" type="imu">
         <always_on>true</always_on>
@@ -113,8 +113,8 @@
         <plugin name="imu" filename="libgazebo_ros_imu_sensor.so"/>
     </sensor>
-  </gazebo>
+  </gazebo> -->
     <!-- 2D Laser Sensor -->
-    <gazebo reference="laser_link">
-      <sensor name="lidar" type="ray">
+    <!-- <gazebo reference="laser_link"> -->
+      <!-- <sensor name="lidar" type="ray">
         <always_on>true</always_on>
         <visualize>true</visualize>
@@ -147,6 +147,6 @@
           <frame_name>laser_link</frame_name>
         </plugin>
-      </sensor>
-      <material>Gazebo/Black</material>
-    </gazebo>
+      </sensor> -->
+      <!-- <material>Gazebo/Black</material> -->
+    <!-- </gazebo> -->
 </robot>
